File: littol.kicad_sch (KiCad schematic)
At the start: 58 parts, among them SW1 SW_Push, SW10 SW_Push, SW11 SW_Push, SW12 SW_Push, SW13 SW_Push, SW14 SW_Push, SW15 SW_Push, SW16 SW_Push, SW17 SW_Push, SW18 SW_Push, SW19 SW_Push, SW2 SW_Push, SW20 SW_Push, SW21 SW_Push, SW22 SW_Push, SW23 SW_Push, SW24 SW_Push, SW25 SW_Push, SW26 SW_Push, SW27 SW_Push, SW28 SW_Push, SW29 SW_Push, SW3 SW_Push, SW4 SW_Push, SW5 SW_Push, SW6 SW_Push, SW7 SW_Push, SW8 SW_Push, SW9 SW_Push

Commit message: added por micron
Parts:
- added U1: ProMicro, symbol promicro:ProMicro
Changed lines of the file:
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@@
+    )
+  )
+  (symbol (lib_id "promicro:ProMicro") (at 212.09 41.91 0) (unit 1)
+    (in_bom yes) (on_board yes) (dnp no) (fields_autoplaced)
+    (property "Reference" "U1" (at 212.09 15.24 0)
+      (effects (font (size 1.524 1.524)))
+    )
+    (property "Value" "ProMicro" (at 212.09 17.78 0)
+      (effects (font (size 1.524 1.524)))
+    )
+    (property "Footprint" "" (at 214.63 68.58 0)
+      (effects (font (size 1.524 1.524)))
+    )
+    (property "Datasheet" "" (at 214.63 68.58 0)
+      (effects (font (size 1.524 1.524)))
+    )
+    (pin "1")
+    (pin "10")
+    (pin "11")
+    (pin "12")
+    (pin "13")
+    (pin "14")
+    (pin "15")
+    (pin "16")
+    (pin "17")
+    (pin "18")
+    (pin "19")
+    (pin "2")
+    (pin "20")
+    (pin "21")
+    (pin "22")
+    (pin "23")
+    (pin "24")
+    (pin "3")
+    (pin "4")
+    (pin "5")
+    (pin "6")
+    (pin "7")
+    (pin "8")
+    (pin "9")
+    (instances
+      (project "littol"
+        (path "/fe1f6a57-af5c-4414-9725-50fa8278502c"
+          (reference "U1") (unit 1)
+        )
+      )
     )
   )

Commit message: started pcb
Parts:
- D1, D10, D11, D12, D13, D14, D15, D16, D17, D18, D19, D2, D20, D21, D22, D23, D24, D25, D26, D27, D28, D29, D3, D4, D5, D6, D7, D8, D9: footprint (none) -> Diode_SMD:D_SOD-123
- SW1, SW10: footprint (none) -> Alps_Solderable:Alps-Solderable-1.5U
- SW11, SW20: footprint (none) -> Alps_Solderable:Alps-Solderable-1.25U
- SW12, SW13, SW14, SW15, SW16, SW17, SW18, SW19, SW2, SW21, SW22, SW23, SW24, SW25, SW26, SW27, SW28, SW3, SW4, SW5, SW6, SW7, SW8, SW9: footprint (none) -> Alps_Solderable:Alps-Solderable-1U
- SW29: footprint (none) -> Alps_Solderable:Alps-Solderable-2U
- U1: footprint (none) -> promicro:ProMicro
